Commit message: reviese something

File: low-level/resources/robots/spot_with_arm_urdf/urdf/spot_with_arm.urdf (robot description, URDF)
Before this commit: robot spot, 20 links, 19 joints
Links:
- link arm0.link_el0: geometry visual mesh filename=../meshes/arm0.link_el0.stl
- link arm0.link_el1: geometry visual mesh filename=../eshes/arm0.link_el1.stl
- link arm0.link_fngr: geometry visual mesh filename=../meshes/arm0.link_fngr.stl
- link arm0.link_sh0: geometry visual mesh filename=../meshes/arm0.link_sh0.stl
- link arm0.link_sh1: geometry visual mesh filename=../meshes/arm0.link_hr0.stl; visual mesh filename=../meshes/arm0.link_sh1.stl
- link arm0.link_wr0: geometry visual mesh filename=../meshes/arm0.link_wr0.stl
- link arm0.link_wr1: geometry visual mesh filename=../meshes/arm0.link_wr1.stl
- link base: geometry collision box size=0.85 0.24 0.18; visual mesh filename=../meshes/base_link_0_geom_visual_mesh.stl
- link fl.hip: geometry visual mesh filename=../meshes/fl_hip_0_geom_visual_mesh.stl
- link fl.lleg: geometry collision cylinder length=0.03 radius=0.033; collision cylinder length=0.35 radius=0.015
- link fl.uleg: geometry collision cylinder length=0.35 radius=0.045; visual mesh filename=../meshes/l_uleg_0_geom_visual_mesh.stl
- link fr.hip: geometry visual mesh filename=../meshes/fr_hip_0_geom_visual_mesh.stl
- link fr.lleg: geometry collision cylinder length=0.03 radius=0.033; collision cylinder length=0.35 radius=0.015
- link fr.uleg: geometry collision cylinder length=0.35 radius=0.045; visual mesh filename=../meshes/r_uleg_0_geom_visual_mesh.stl
- link hl.hip: geometry visual mesh filename=../meshes/hl_hip_0_geom_visual_mesh.stl
- link hl.lleg: geometry collision cylinder length=0.03 radius=0.033; collision cylinder length=0.35 radius=0.015
- link hl.uleg: geometry collision cylinder length=0.35 radius=0.045; visual mesh filename=../meshes/l_uleg_0_geom_visual_mesh.stl
- link hr.hip: geometry visual mesh filename=../meshes/hr_hip_0_geom_visual_mesh.stl
- link hr.lleg: geometry collision cylinder length=0.03 radius=0.033; collision cylinder length=0.35 radius=0.015
- link hr.uleg: geometry collision cylinder length=0.35 radius=0.045; visual mesh filename=../meshes/r_uleg_0_geom_visual_mesh.stl
Joints:
- removed joint fl.hx
- removed joint fl.hy
- removed joint fl.kn
- removed joint fr.hx
- removed joint fr.hy
- removed joint fr.kn
- removed joint hl.hx
- removed joint hl.hy
- removed joint hl.kn
- removed joint hr.hx
- removed joint hr.hy
- removed joint hr.kn
- added joint fl.hx_joint: type revolute, parent base, child fl.hip, origin xyz=0.29785 0.05500 0.00000, axis 1 0 0, limit lower=-0.785398 upper=0.785398 effort=45 velocity=100
- added joint fl.hy_joint: type revolute, parent fl.hip, child fl.uleg, origin xyz=0.0 0.110945 0.0, axis 0 1 0, limit lower=-0.898845 upper=2.295108 effort=45 velocity=100
- added joint fl.kn_joint: type revolute, parent fl.uleg, child fl.lleg, origin xyz=0.025 0.000 -0.3205, axis 0 1 0, limit lower=-2.7929 upper=-0.2471 effort=115 velocity=100
- added joint fr.hx_joint: type revolute, parent base, child fr.hip, origin xyz=0.29785 -0.05500 0.00000, axis 1 0 0, limit lower=-0.785398 upper=0.785398 effort=45 velocity=100
- added joint fr.hy_joint: type revolute, parent fr.hip, child fr.uleg, origin xyz=0.0 -0.110945 0.0, axis 0 1 0, limit lower=-0.898845 upper=2.295108 effort=45 velocity=100
- added joint fr.kn_joint: type revolute, parent fr.uleg, child fr.lleg, origin xyz=0.025 0.000 -0.3205, axis 0 1 0, limit lower=-2.7929 upper=-0.2471 effort=115 velocity=100
- added joint hl.hx_joint: type revolute, parent base, child hl.hip, origin xyz=-0.29785 0.05500 0.00000, axis 1 0 0, limit lower=-0.785398 upper=0.785398 effort=45 velocity=100
- added joint hl.hy_joint: type revolute, parent hl.hip, child hl.uleg, origin xyz=0.0 0.110945 0.0, axis 0 1 0, limit lower=-0.898845 upper=2.295108 effort=45 velocity=100
- added joint hl.kn_joint: type revolute, parent hl.uleg, child hl.lleg, origin xyz=0.025 0.000 -0.3205, axis 0 1 0, limit lower=-2.7929 upper=-0.2471 effort=115 velocity=100
- added joint hr.hx_joint: type revolute, parent base, child hr.hip, origin xyz=-0.29785 -0.05500 0.00000, axis 1 0 0, limit lower=-0.785398 upper=0.785398 effort=45 velocity=100
- added joint hr.hy_joint: type revolute, parent hr.hip, child hr.uleg, origin xyz=0.0 -0.110945 0.0, axis 0 1 0, limit lower=-0.898845 upper=2.295108 effort=45 velocity=100
- added joint hr.kn_joint: type revolute, parent hr.uleg, child hr.lleg, origin xyz=0.025 0.000 -0.3205, axis 0 1 0, limit lower=-2.7929 upper=-0.2471 effort=115 velocity=100
